File: UCubeSat-EPS.kicad_sch (KiCad schematic)
At the start: 0 parts

Commit message: update
Other:
- note added: "LALALALALA, UPDATING SCHEMATIC. WILL IT UPDATE??? WHO KNOWS???"
Changed lines of the file:
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@@
 	(generator_version "9.0")
 	(paper "A4")
+	(text "LALALALALA, UPDATING SCHEMATIC. WILL IT UPDATE??? WHO KNOWS???"
+		(exclude_from_sim no)
+		(at 110.744 122.936 0)
+		(effects
+			(font
+				(size 1.27 1.27)
+			)
+		)
+	)
 	(sheet_instances
 		(path "/"
